Commit message: Changed the Scan Range

File: saclebot_description/urdf/saclebot_description.urdf (robot description, URDF)
Before this commit: robot saclebot, 34 links, 33 joints
Joints:
- joint RP_LiDAR_A3M1_joint: origin xyz=0.15749 -0.0096 0.126 rpy=0 0 -3.1416 -> xyz=0.15749 -0.0096 0.126 rpy=0 0 0

Commit message: Added Changed meshes in urdf!

File: saclebot_description/urdf/saclebot_description.urdf (robot description, URDF)
Before this commit: robot saclebot, 34 links, 33 joints
Links:
- link R1_link: geometry collision mesh filename=package://saclebot_description/meshes/R1_link.dae; visual mesh filename=package://saclebot_description/meshes/R1_link.dae
- link R2_link: geometry collision mesh filename=package://saclebot_description/meshes/R2_link.dae; visual mesh filename=package://saclebot_description/meshes/R2_link.dae
- link R3_link: geometry collision mesh filename=package://saclebot_description/meshes/R3_link.dae; visual mesh filename=package://saclebot_description/meshes/R3_link.dae
- link RP_LiDAR_A3M1_link: geometry collision mesh filename=package://saclebot_description/meshes/RP_LiDAR_A3M1_link.dae; visual mesh filename=package://saclebot_description/meshes/RP_LiDAR_A3M1_link.dae
- link base_link: geometry collision mesh filename=package://saclebot_description/meshes/base_link.dae; visual mesh filename=package://saclebot_description/meshes/base_link.dae
- link frontLeftWheel_link: geometry collision mesh filename=package://saclebot_description/meshes/frontLeftWheel_link.d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; visual mesh filename=package://saclebot_description/meshes/frontLeftWheel_link.d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
- link mop_link: geometry collision mesh filename=package://saclebot_description/meshes/mop_link.dae; visual mesh filename=package://saclebot_description/meshes/mop_link.dae
- link rearLeftWheel_link: geometry collision mesh filename=package://saclebot_description/meshes/rearLeftWheel_link.dae; visual mesh filename=package://saclebot_description/meshes/rearLeftWheel_link.dae
- link rearRightWheel_link: geometry collision mesh filename=package://saclebot_description/meshes/rearRightWheel_link.d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; visual mesh filename=package://saclebot_description/meshes/rearRightWheel_link.d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
- link shoulder_link: geometry collision mesh filename=package://saclebot_description/meshes/shoulder_link.dae; visual mesh filename=package://saclebot_description/meshes/shoulder_link.dae
- link slider_link: geometry collision mesh filename=package://saclebot_description/meshes/slider_link.dae; visual mesh filename=package://saclebot_description/meshes/slider_link.dae
Joints:
- joint R3_joint: limit lower=-1.5708 upper=3.1416 effort=2 velocity=2 -> lower=0.0 upper=3.1416 effort=2 velocity=2

Commit message: Added possibility to relocate the robot!

File: saclebot_description/urdf/saclebot_description.urdf (robot description, URDF)
Before this commit: robot saclebot, 34 links, 33 joints
Links:
- link base_link: mass 4.57525 -> 1.1438125
- link base_manipulator: mass 1.0364 -> 0.5182
- link shoulder_link: mass 0.6828 -> 0.3414
